File: PC218/PC218.kicad_sch (KiCad schematic)
At the start: 106 parts, among them J1 PC218_BoardEdge_44pin, Q1 BC848W, Q10 BC848W, Q11 BC848W, Q12 BC848W, Q13 BC848W, Q14 BC848W, Q15 BC848W, Q16 BC848W, Q17 BC848W, Q18 BC848W, Q19 BC848W, Q2 BC848W, Q20 BC848W, Q21 BC848W, Q22 BC848W, Q23 BC848W, Q24 BC848W, Q25 BC848W, Q26 BC848W, Q27 BC848W, Q28 BC848W, Q29 BC848W, Q3 BC848W, Q30 BC848W, Q31 BC848W, Q32 BC848W, Q33 BC848W, Q34 BC848W, Q35 BC848W, Q36 BC848W, Q37 BC848W, Q38 BC848W, Q39 BC848W, Q4 BC848W, Q40 BC848W, Q41 BC848W, Q42 BC848W, Q43 BC848W, Q44 BC848W, Q45 BC848W, Q5 BC848W, Q6 BC848W, Q7 BC848W, Q8 BC848W, Q9 BC848W

Commit message: PC218 Rev 1.1
Fixed disconnected ground plane resulting in two buffers being unpowered
Moved silkscreen to front, add OSHW logo
Move symbols and footprints to shared library
Update edge connector footprint to use a more sane orientation
Parts:
- J1: footprint keithley_615_part_library:PC218_Edge_Connector -> footprints:PC218_Edge_Connector; symbol keithley_615_sym_library:PC218_BoardEdge_44pin -> lib_symbols:PC218_BoardEdge_44pin
Other:
- company: (none) -> Peter Farley
- title: (none) -> Keithley 615 PC218 Replacement Board
Changed lines of the file:
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@@
 (kicad_sch (version 20211123) (generator eeschema)
   (paper "A3")
+  (title_block
+    (title "Keithley 615 PC218 Replacement Board")
+    (date "2023-01-10")
+    (rev "1.0")
+    (company "Peter Farley")
+    (comment 1 "Rev 1: Initial design")
+  )
   (junction (at 49.53 179.07) (diameter 0) (color 0 0 0 0)
   )
@@
     (pin "2")
   )
-  (symbol (lib_id "keithley_615_sym_library:PC218_BoardEdge_44pin") (at 229.87 19.05 0) (unit 1)
+  (symbol (lib_id "lib_symbols:PC218_BoardEdge_44pin") (at 229.87 19.05 0) (unit 1)
     (in_bom yes) (on_board yes) (fields_autoplaced)
     (property "Reference" "J1" (id 0) (at 229.235 15.24 0))
     (property "Value" "PC218_BoardEdge_44pin" (id 1) (at 229.235 17.78 0))
-    (property "Footprint" "keithley_615_part_library:PC218_Edge_Connector" (id 2) (at 228.6 19.05 0)
+    (property "Footprint" "footprints:PC218_Edge_Connector" (id 2) (at 228.6 19.05 0)
       (effects (font (size 1.27 1.27)) hide)
     )
@@
     )
     (path "/0b3e7a7c-ceb5-44cc-8e1c-4b20ca10ed23"
-      (reference "J1") (unit 1) (value "PC218_BoardEdge_44pin") (footprint "keithley_615_part_library:PC218_Edge_Connector")
+      (reference "J1") (unit 1) (value "PC218_BoardEdge_44pin") (footprint "footprints:PC218_Edge_Connector")
     )
     (path "/4446f63d-df20-417e-add3-680a46456664"
