File: 50PinTestBoard/50PinTestBoard.kicad_pcb (KiCad board)
At the start: 2 copper layers, 78 x 3.1 mm, 158 parts, among them J1 Keithley_50-Pin_Connector, Q1 BC848W, Q10 BC848W, Q11 BC848W, Q12 BC848W, Q13 BC848W, Q14 BC848W, Q15 BC848W, Q16 BC848W, Q17 BC848W, Q18 BC848W, Q19 BC848W, Q2 BC848W, Q20 BC848W, Q21 BC848W, Q22 BC848W, Q23 BC848W, Q24 BC848W, Q25 BC848W, Q3 BC848W, Q4 BC848W, Q5 BC848W, Q6 BC848W, Q7 BC848W, Q8 BC848W, Q9 BC848W, SW1 SW_SPST, SW2 SW_SPST, SW3 SW_Push

Commit message: 50PinTestBoard: Rev 1.0
Parts:
- removed the D16 at (205.4, 55.2)
- removed the D17 at (210.6, 60.8)
- removed the Q16 at (192.3, 52.8)
- removed the Q17 at (185.7, 68.8)
- removed the R31 at (217.2, 75.8)
- removed the R32 at (230.7, 62.2)
- removed the R41 at (202.0, 67.4)
- removed the R42 at (218.1, 70.8)
- removed the TP10 at (194.4, 63.9)
- removed the TP11 at (229.7, 48.2)
- removed the TP12 at (217.6, 57.5)
- removed the TP13 at (254.0, 48.2)
- removed the TP14 at (237.8, 54.9)
- removed the TP15 at (209.5, 53.4)
- removed the TP25 at (189.9, 67.6)
- removed the TP26 at (213.5, 53.4)
- removed the TP27 at (250.0, 48.2)
- removed the TP28 at (205.4, 51.9)
- removed the TP29 at (217.6, 53.4)
- removed the TP3 at (189.9, 71.6)
- removed the TP30 at (229.7, 54.9)
- removed the TP31 at (233.8, 48.2)
- removed the TP32 at (241.9, 58.6)
- removed the TP4 at (245.9, 53.4)
- removed the TP5 at (250.0, 52.3)
- removed the TP6 at (198.4, 63.9)
- removed the TP7 at (225.7, 54.9)
- removed the TP8 at (221.6, 48.2)
- removed the TP9 at (233.8, 52.3)
- added REF**: OSHW-Logo_7.5x8mm_SilkScreen, Symbol:OSHW-Logo_7.5x8mm_SilkScreen, B.Cu at (70.9, 120.5)
- added REF**: KiCad-Logo2_5mm_SilkScreen, Symbol:KiCad-Logo2_5mm_SilkScreen, B.Cu at (56.2, 121.0)
- added TP1: TestPoint, TestPoint:TestPoint_THTPad_2.0x2.0mm_Drill1.0mm, F.Cu at (35.9, 47.8)
- TP10: renamed from TP6; footprint TestPoint:TestPoint_Pad_2.0x2.0mm -> TestPoint:TestPoint_THTPad_2.0x2.0mm_Drill1.0mm
- TP11: renamed from TP5; footprint TestPoint:TestPoint_Pad_2.0x2.0mm -> TestPoint:TestPoint_THTPad_2.0x2.0mm_Drill1.0mm
- TP12: renamed from TP4; footprint TestPoint:TestPoint_Pad_2.0x2.0mm -> TestPoint:TestPoint_THTPad_2.0x2.0mm_Drill1.0mm
- TP13: renamed from TP3; footprint TestPoint:TestPoint_Pad_2.0x2.0mm -> TestPoint:TestPoint_THTPad_2.0x2.0mm_Drill1.0mm
- TP14: renamed from TP2; footprint TestPoint:TestPoint_Pad_2.0x2.0mm -> TestPoint:TestPoint_THTPad_2.0x2.0mm_Drill1.0mm
- TP15: renamed from TP1; footprint TestPoint:TestPoint_Pad_2.0x2.0mm -> TestPoint:TestPoint_THTPad_2.0x2.0mm_Drill1.0mm
- TP2, TP8: footprint TestPoint:TestPoint_Pad_2.0x2.0mm -> TestPoint:TestPoint_THTPad_2.0x2.0mm_Drill1.0mm
- TP23: renamed from TP15; footprint TestPoint:TestPoint_Pad_2.0x2.0mm -> TestPoint:TestPoint_THTPad_2.0x2.0mm_Drill1.0mm
- TP24: renamed from TP14; footprint TestPoint:TestPoint_Pad_2.0x2.0mm -> TestPoint:TestPoint_THTPad_2.0x2.0mm_Drill1.0mm
- TP25: renamed from TP32; footprint TestPoint:TestPoint_Pad_2.0x2.0mm -> TestPoint:TestPoint_THTPad_2.0x2.0mm_Drill1.0mm
- TP26: renamed from TP31; footprint TestPoint:TestPoint_Pad_2.0x2.0mm -> TestPoint:TestPoint_THTPad_2.0x2.0mm_Drill1.0mm
- TP27: renamed from TP30; footprint TestPoint:TestPoint_Pad_2.0x2.0mm -> TestPoint:TestPoint_THTPad_2.0x2.0mm_Drill1.0mm
- TP28: renamed from TP29; footprint TestPoint:TestPoint_Pad_2.0x2.0mm -> TestPoint:TestPoint_THTPad_2.0x2.0mm_Drill1.0mm
- TP29: renamed from TP28; footprint TestPoint:TestPoint_Pad_2.0x2.0mm -> TestPoint:TestPoint_THTPad_2.0x2.0mm_Drill1.0mm
- TP3: renamed from TP13; footprint TestPoint:TestPoint_Pad_2.0x2.0mm -> TestPoint:TestPoint_THTPad_2.0x2.0mm_Drill1.0mm
- TP30: renamed from TP27; footprint TestPoint:TestPoint_Pad_2.0x2.0mm -> TestPoint:TestPoint_THTPad_2.0x2.0mm_Drill1.0mm
- TP31: renamed from TP26; footprint TestPoint:TestPoint_Pad_2.0x2.0mm -> TestPoint:TestPoint_THTPad_2.0x2.0mm_Drill1.0mm
- TP32: renamed from TP25; footprint TestPoint:TestPoint_Pad_2.0x2.0mm -> TestPoint:TestPoint_THTPad_2.0x2.0mm_Drill1.0mm
- TP4: renamed from TP12; footprint TestPoint:TestPoint_Pad_2.0x2.0mm -> TestPoint:TestPoint_THTPad_2.0x2.0mm_Drill1.0mm
- TP5: renamed from TP11; footprint TestPoint:TestPoint_Pad_2.0x2.0mm -> TestPoint:TestPoint_THTPad_2.0x2.0mm_Drill1.0mm
- TP6: renamed from TP10; footprint TestPoint:TestPoint_Pad_2.0x2.0mm -> TestPoint:TestPoint_THTPad_2.0x2.0mm_Drill1.0mm
- TP7: renamed from TP9; footprint TestPoint:TestPoint_Pad_2.0x2.0mm -> TestPoint:TestPoint_THTPad_2.0x2.0mm_Drill1.0mm
- TP9: renamed from TP7; footprint TestPoint:TestPoint_Pad_2.0x2.0mm -> TestPoint:TestPoint_THTPad_2.0x2.0mm_Drill1.0mm
- moved TP2 241.9 mm to (35.9, 52.2), turned to -90 degrees
- moved Q23 220.8 mm to (70.4, 126.7)
- moved TP25 219.5 mm to (63.2, 87.5)
- moved TP26 216.4 mm to (63.2, 97.0)
- moved Q22 213.3 mm to (70.4, 122.3)
- moved TP28 210.9 mm to (63.2, 109.2)
- moved TP31 208.7 mm to (63.2, 122.2)
- moved TP27 207.6 mm to (63.2, 101.5)
- moved TP29 206.2 mm to (63.2, 113.5)
- moved Q17 205.6 mm to (70.4, 97.0)
- moved D6 204.0 mm to (46.9, 92.4)
- moved D9 202.1 mm to (46.9, 105.9)
- moved TP30 201.1 mm to (63.2, 117.8)
- moved TP32 200.6 mm to (63.2, 126.8)
- moved D7 200.5 mm to (46.9, 96.9)
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- renumbered D13 to D1, D4 to D10, D3 to D11, D2 to D12, D1 to D13, D15 to D14, D14 to D15, D18 to D16, D19 to D17, D20 to D18, D21 to D19, D12 to D2, D22 to D20, D23 to D21, D24 to D22, D25 to D23, D11 to D3, D10 to D4, D9 to D5, D8 to D6, D6 to D8, D5 to D9, Q13 to Q1, Q4 to Q10, Q3 to Q11, Q2 to Q12, Q1 to Q13, Q15 to Q14, Q14 to Q15, Q18 to Q16, Q19 to Q17, Q20 to Q18, Q21 to Q19, Q12 to Q2, Q22 to Q20, Q23 to Q21, Q24 to Q22, Q25 to Q23, Q11 to Q3, Q10 to Q4, Q9 to Q5, Q8 to Q6, Q6 to Q8, Q5 to Q9, R25 to R1, R16 to R10, R15 to R11, R14 to R12, R28 to R14, R12 to R15, R11 to R16, R10 to R17, R9 to R18, R8 to R19, R24 to R2, R7 to R20, R6 to R21, R5 to R22, R4 to R23, R3 to R24, R2 to R25, R1 to R26, R26 to R28, R33 to R29, R23 to R3, R34 to R30, R35 to R31, R36 to R32, R37 to R33, R38 to R34, R39 to R35, R40 to R36, R30 to R37, R29 to R38, R43 to R39, R22 to R4, R44 to R40, R45 to R41, R46 to R42, R47 to R43, R48 to R44, R49 to R45, R50 to R46, R21 to R5, R20 to R6, R19 to R7, R18 to R8, R17 to R9, SW3 to SW1, SW1 to SW2, SW2 to SW3, TP24 to TP22, TP22 to TP33, TP23 to TP34
Connections:
- TP16 pad 1: Net-(J1-Pad42) -> Net-(J1-Pad14)
- TP17 pad 1: Net-(J1-Pad18) -> Net-(J1-Pad25)
- TP18 pad 1: Net-(J1-Pad14) -> Net-(J1-Pad18)
- TP19 pad 1: GND -> Net-(J1-Pad42)
- TP2 pad 1: Net-(Q2-Pad1) -> +5V
- TP21 pad 1: Net-(J1-Pad25) -> GND
Routing:
- net +5V: track 0.00 -> 196.7 mm, vias 0 -> 4
- net Net-(J1-Pad30): track 0.00 -> 83.7 mm
- net Net-(J1-Pad26): track 0.00 -> 80.7 mm
- net Net-(J1-Pad14): track 0.00 -> 80.5 mm
- net Net-(J1-Pad31): track 0.00 -> 78.7 mm
- net Net-(J1-Pad28): track 0.00 -> 78.0 mm
- net Net-(J1-Pad7): track 0.00 -> 76.5 mm
- net Net-(J1-Pad29): track 0.00 -> 71.7 mm
- net Net-(J1-Pad6): track 0.00 -> 70.3 mm
- net Net-(J1-Pad5): track 0.00 -> 69.2 mm
- net Net-(J1-Pad1): track 0.00 -> 68.7 mm
- net Net-(J1-Pad27): track 0.00 -> 66.9 mm
- net Net-(J1-Pad2): track 0.00 -> 66.0 mm
- net Net-(J1-Pad46): track 0.00 -> 65.4 mm
- net Net-(J1-Pad4): track 0.00 -> 64.7 mm
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- added copper zone on B.Cu, net GND
- added copper zone on F.Cu, net GND
Other:
- board size 78 x 3.1 mm -> 75 x 88 mm
- board text added: "+15V"
- board text added: "+3.6V"
- board text added: "+5V"
- board text added: "-15V"
- board text added: "Data 1e0"
- board text added: "Data 1e1"
- board text added: "Data 1e2"
- board text added: "Data 1e3"
- board text added: "Data 2e0"
- board text added: "Data 2e1"
- board text added: "Data 2e2"
- board text added: "Data 4e0"
- board text added: "Data 4e1"
- board text added: "Data 4e2"
- board text added: "Data 8e0"
- board text added: "Data 8e1"
- board text added: "Data 8e2"
- board text added: "GND"
- board text added: "Hold1"
- board text added: "Hold2"
- board text added: "Keithley 615 50-Pin Test Board V1.0 Peter Farley, 2013"
- board text added: "Overload"
- board text added: "Polarity"
- board text added: "Print"
- board text added: "Range 1e0"
- board text added: "Range 1e1"
- board text added: "Range 2e0"
- board text added: "Range 4e0"
- board text added: "Range 8e0"
- board text added: "Ref. Hi"
- board text added: "Ref. Lo"
- board text added: "Sensitivity 1e0"
- board text added: "Sensitivity 2e0"
- board text added: "Trigger"

Commit message: 50PinTestBoard: Rev 1.1
Made screw holes for connector foot print plated through-holes.
Parts:
- added R47: 0, Resistor_SMD:R_0603_1608Metric, B.Cu at (102.0, 50.5)
- added R48: 0, Resistor_SMD:R_0603_1608Metric, B.Cu at (102.0, 125.5)
Routing:
- net Net-(J1-Pad52): track 0.00 -> 4.78 mm
- net Net-(J1-Pad51): track 0.00 -> 4.78 mm

Commit message: 50PinTestBoard: Fix year
Other:
- board text added: "Keithley 615 50-Pin Test Board V1.0 Peter Farley, 2023"
- board text removed: "Keithley 615 50-Pin Test Board V1.0 Peter Farley, 2013"
Changed lines of the file:
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@@
   (title_block
     (title "Keithley 615 50-Pin Test Board")
-    (date "2023-01-21")
+    (date "2023-02-03")
     (rev "1.1")
     (company "Peter Farley")
@@
   (gr_line (start 107.434302 46) (end 107.434302 130) (layer "Edge.Cuts") (width 0.1))
   (gr_line (start 35.434302 44) (end 105.434302 44) (layer "Edge.Cuts") (width 0.1))
-  (gr_text "Keithley 615 50-Pin Test Board V1.0\nPeter Farley, 2013" (at 46.6 61.5 90) (layer "B.SilkS")
+  (gr_text "Keithley 615 50-Pin Test Board V1.0\nPeter Farley, 2023" (at 46.6 61.5 90) (layer "B.SilkS")
     (effects (font (size 2 2) (thickness 0.2)) (justify left mirror))
   )

Commit message: 50PinTestBoard: Rev 1.2
Fix orientation of connector footprint
 - Moved connector to bottom of board to avoid re-routing entire board.
Update resistor value(s).
Add Digi-Key links for parts.
Parts:
- J1: moved to B.Cu
- R47: renamed from R48; moved to F.Cu
- R48: renamed from R47; moved to F.Cu
- moved R47 75.0 mm to (102.0, 50.5)
- moved R48 75.0 mm to (102.0, 125.5)
- turned J1 to 90 degrees
- renumbered R5 to R1, R7 to R2, R34 to R27, R27 to R28, R28 to R29, R1 to R3, R29 to R30, R30 to R31, R31 to R32, R32 to R33, R33 to R34, R2 to R4, R3 to R5, R4 to R6, R6 to R7
Other:
- board text added: "Keithley 615 50-Pin Test Board V1.2 Peter Farley, 2023"
- board text removed: "Keithley 615 50-Pin Test Board V1.0 Peter Farley, 2023"
