File: InterfaceBoard/InterfaceBoard.kicad_pcb (KiCad board)
At the start: 2 copper layers, 100 x 86 mm, 186 parts, among them J1 SPI, J2 I2C, J3 Keithley_50-Pin_Connector, J4 SWD, J5 UART, J6 USB_B, J7 RS232, J8 DB9_Female_MountingHoles, P1 RB1-125BAG1A, Q1 BC848W, Q2 BC848W, Q3 BC848W, Q4 BC856W, SW1 PTS810, SW2 PTS810, U1 W5500, U2 STM32G0B1RET, U3 AP62250Z6, U4 FT231XQ, U5 MAX3232, Y1 25 MHz, Y2 24 MHz, Y3 32.768 kHz

Commit message: InterfaceBoard: Rev 1.0
Parts:
- removed the R35 at (116.8, 74.8)
- removed the R36 at (118.3, 74.8)
- removed the R37 at (119.8, 74.8)
- added J5: Conn_02x03_Odd_Even, Connector_PinHeader_1.27mm:PinHeader_2x03_P1.27mm_Vertical, F.Cu at (117.0, 75.3)
- renumbered J5 to J6, J6 to J7, J7 to J8, J8 to J9, R38 to R35, R39 to R36, R40 to R37, R41 to R38, R42 to R39, R43 to R40, R44 to R41, R45 to R42, R46 to R43, R47 to R44, R48 to R45, R49 to R46, R50 to R47, R51 to R48, R52 to R49, R53 to R50, R54 to R51, R55 to R52, R56 to R53, R57 to R54, R58 to R55, R59 to R56, R60 to R57, R61 to R58, R62 to R59, R63 to R60, R64 to R61, R65 to R62, R66 to R63, R67 to R64, R68 to R65, R69 to R66, R70 to R67, R71 to R68, R72 to R69, R73 to R70, R74 to R71, R75 to R72, R76 to R73, R77 to R74, R78 to R75, R79 to R76, R80 to R77, R81 to R78, R82 to R79, R83 to R80, R84 to R81, R85 to R82, R86 to R83, R87 to R84, R88 to R85, R89 to R86, R90 to R87, R91 to R88, R92 to R89, R93 to R90, R94 to R91
Routing:
- net +15V: track 97.0 -> 99.7 mm, vias 3 -> 2
Other:
- board text added: "Keithley 615 Interface Board v1.0 Peter Farley, 2023"
- board text removed: "Keithley 615 Interface Board Peter Farley, 2023"
- board text removed: "Routed Ethernet differential pairs assuming 2-layer Redo if switching to 4-layer board"
- board text removed: "TODO: Add chassis ground, and pour under RJ45 jack, but not under rx/tx pins."
