File: InterfaceBoard/50pin.kicad_sch (KiCad schematic)
At the start: 55 parts, among them J3 Keithley_50-Pin_Connector, Q1 BC848W, Q2 BC848W, Q3 BC848W

Commit message: InterfaceBoard: Rev 1.0
Parts:
- renumbered Q2 to Q1, Q1 to Q2, R62 to R10, R73 to R11, R64 to R12, R63 to R13, R65 to R14, R61 to R18, R72 to R19, R60 to R20, R71 to R21, R52 to R22, R37 to R23, R59 to R25, R70 to R26, R58 to R27, R69 to R28, R56 to R30, R67 to R31, R57 to R33, R68 to R34, R55 to R35, R66 to R36, R51 to R38, R36 to R39, R50 to R41, R35 to R42, R47 to R43, R32 to R44, R49 to R45, R34 to R46, R46 to R47, R31 to R48, R48 to R49, R33 to R50, R43 to R55, R28 to R56, R45 to R58, R30 to R59, R42 to R60, R27 to R61, R44 to R62, R29 to R63, R39 to R65, R24 to R66, R41 to R68, R26 to R69, R38 to R72, R23 to R73, R40 to R74, R25 to R75, R54 to R80, R53 to R91
Other:
- company: (none) -> Peter Farley
- title: (none) -> Kiethley 615 Interface Board

Commit message: InterfaceBoard: Add BOM
Parts:
- J3: DigiKey (none) -> https://www.digikey.com/en/products/detail/norcomp-inc/112-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
- R10, R18, R20, R22, R25, R27, R30, R33, R35, R38, R41, R43, R45, R47, R49, R55, R58, R60, R62, R65, R68, R72, R74, R80, R91: DigiKey (none) -> https://www.digikey.com/en/products/detail/walsin-technolog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
- R11, R19, R21, R23, R26, R28, R31, R34, R36, R39, R42, R44, R46, R48, R50, R56, R59, R61, R63, R66, R69, R73, R75: DigiKey (none) -> https://www.digikey.com/en/products/detail/stackpole-electr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
- R12, R13, R14: DigiKey (none) -> https://www.digikey.com/en/products/detail/yageo/RC0603FR-1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
