File: InterfaceBoard/MCU.kicad_sch (KiCad schematic)
At the start: 13 parts, among them J4 SWD, U2 STM32G0B1RET, Y2 24 MHz, Y3 32.768 kHz

Commit message: InterfaceBoard: Add BOM
Parts:
- C11: DigiKey (none) -> https://www.digikey.com/en/products/detail/w%C3%BCrth-elekt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
- C30, C31, R86: DigiKey (none) -> https://www.digikey.com/en/products/detail/walsin-technolog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
- C32, C33: DigiKey (none) -> https://www.digikey.com/en/products/detail/samsung-electro-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
- J4: now left out of the parts list
- R16: DigiKey https://www.digikey.com/ordering/shoppingcart -> https://www.digikey.com/en/products/detail/stackpole-electr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
- U2: DigiKey (none) -> https://www.digikey.com/en/products/detail/stmicroelectroni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
Changed lines of the file:
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@@
+      (effects (font (size 1.27 1.27)) hide)
+    )
+    (property "DigiKey" "https://www.digikey.com/en/products/detail/samsung-electro-mechanics/CL10B104KB8NNWC/3887593" (id 4) (at 181.61 60.96 0)
       (effects (font (size 1.27 1.27)) hide)
     )
@@
       (effects (font (size 1.27 1.27)) hide)
     )
+    (property "DigiKey" "https://www.digikey.com/en/products/detail/walsin-technology-corporation/0603N220J500CT/9355000" (id 4) (at 181.61 102.87 0)
+      (effects (font (size 1.27 1.27)) hide)
+    )
     (pin "1")
     (pin "2")
@@
       (effects (font (size 1.27 1.27)) hide)
     )
+    (property "DigiKey" "https://www.digikey.com/en/products/detail/walsin-technology-corporation/WR06X000-PTL/5978108" (id 4) (at 181.61 57.15 0)
+      (effects (font (size 1.27 1.27)) hide)
+    )
     (pin "1")
     (pin "2")
@@
       (effects (font (size 1.27 1.27)) hide)
     )
-    (property "DigiKey" "https://www.digikey.com/ordering/shoppingcart" (id 4) (at 162.56 140.97 90)
+    (property "DigiKey" "https://www.digikey.com/en/products/detail/stackpole-electronics-inc/RMCF0603FT1K60/1761204" (id 4) (at 162.56 140.97 90)
       (effects (font (size 1.27 1.27)) hide)
     )
@@
       (effects (font (size 1.27 1.27)) hide)
     )
+    (property "DigiKey" "https://www.digikey.com/en/products/detail/samsung-electro-mechanics/CL10B104KB8NNWC/3887593" (id 4) (at 228.6 137.16 0)
+      (effects (font (size 1.27 1.27)) hide)
+    )
     (pin "1")
     (pin "2")
   )
   (symbol (lib_id "Connector:Conn_ARM_JTAG_SWD_10") (at 248.92 53.34 0) (unit 1)
-    (in_bom yes) (on_board yes) (fields_autoplaced)
+    (in_bom no) (on_board yes) (fields_autoplaced)
     (property "Reference" "J4" (id 0) (at 237.49 52.0699 0)
       (effects (font (size 1.27 1.27)) (justify right))
@@
       (effects (font (size 1.27 1.27)) hide)
     )
-    (property "Datasheet" "~" (id 3) (at 236.22 137.16 0)
+    (property "Datasheet" "https://www.we-online.com/components/products/datasheet/865230642008.pdf" (id 3) (at 236.22 137.16 0)
+      (effects (font (size 1.27 1.27)) hide)
+    )
+    (property "DigiKey" "https://www.digikey.com/en/products/detail/w%C3%BCrth-elektronik/865230642008/5727868" (id 4) (at 236.22 137.16 0)
       (effects (font (size 1.27 1.27)) hide)
     )
@@
     )
     (property "Datasheet" "" (id 3) (at 130.81 54.61 0)
+      (effects (font (size 1.27 1.27)) hide)
+    )
+    (property "DigiKey" "https://www.digikey.com/en/products/detail/stmicroelectronics/STM32G0B1RET6/13693663" (id 4) (at 137.16 54.61 0)
       (effects (font (size 1.27 1.27)) hide)
     )
@@
       (effects (font (size 1.27 1.27)) hide)
     )
+    (property "DigiKey" "https://www.digikey.com/en/products/detail/walsin-technology-corporation/0603N220J500CT/9355000" (id 4) (at 181.61 110.49 0)
+      (effects (font (size 1.27 1.27)) hide)
+    )
