File: InterfaceBoard/USB.kicad_sch (KiCad schematic)
At the start: 19 parts, among them J2 USB_B, U2 FT231XS

Commit message: InterfaceBoard: Add RS-232/DE-9
Parts:
- U2: value FT231XS -> FT231XQ; footprint Package_SO:SSOP-20_3.9x8.7mm_P0.635mm -> Package_DFN_QFN:QFN-20-1EP_4x4mm_P0.5mm_EP2.5x2.5mm; symbol Interface_USB:FT231XS -> Interface_USB:FT231XQ
Connections:
- net GND: now also U2.21 (GND), U2.3 (GND); no longer U2.16 (GND), U2.6 (GND)
- net USB_UART_CTS: now also U2.6 (~{CTS}); no longer U2.9 (~{CTS})
- net USB_UART_RTS: now also U2.19 (~{RTS}); no longer U2.2 (~{RTS})
- net USB_UART_RX: now also U2.1 (RXD); no longer U2.4 (RXD)
- net USB_UART_TX: now also U2.17 (TXD); no longer U2.20 (TXD)
- net V_USB: now also U2.12 (VCC); no longer U2.15 (VCC)
- net USBB_D-: now reaches C18.1, J2.2 (D-), R18.1, R20.1, R76.1
- net USBB_D+: now reaches C17.1, J2.3 (D+), R17.1, R19.1, R75.1
- net FTDI_VCC: now reaches C20.1, R21.2, R22.2
- net FTDI_VCC: now also U2.10 (3V3OUT), U2.11 (~{RESET}), U2.20 (VCCIO); no longer U2.13 (3V3OUT), U2.14 (~{RESET}), U2.3 (VCCIO)
- net FTDI_RX_LED: now reaches D3.1 (K)
- net FTDI_RX_LED: now also U2.14 (CBUS1); no longer U2.17 (CBUS1)
- net FTDI_D+: now reaches R19.2
- net FTDI_D+: now also U2.8 (USBDP); no longer U2.11 (USBDP)
- net FTDI_TX_LED: now reaches D4.1 (K)
- net FTDI_TX_LED: now also U2.7 (CBUS2); no longer U2.10 (CBUS2)
- net FTDI_D-: now reaches R20.2
- net FTDI_D-: now also U2.9 (USBDM); no longer U2.12 (USBDM)
Changed lines of the file:
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@@
     (stroke (width 0) (type default) (color 0 0 0 0))
   )
-  (wire (pts (xy 134.62 76.2) (xy 140.97 76.2))
+  (wire (pts (xy 132.08 76.2) (xy 140.97 76.2))
     (stroke (width 0) (type default) (color 0 0 0 0))
   )
@@
     (stroke (width 0) (type default) (color 0 0 0 0))
   )
-  (wire (pts (xy 123.19 72.39) (xy 134.62 72.39))
-    (stroke (width 0) (type default) (color 0 0 0 0))
-  )
-  (wire (pts (xy 134.62 72.39) (xy 134.62 76.2))
+  (wire (pts (xy 123.19 72.39) (xy 132.08 72.39))
+    (stroke (width 0) (type default) (color 0 0 0 0))
+  )
+  (wire (pts (xy 132.08 72.39) (xy 132.08 76.2))
     (stroke (width 0) (type default) (color 0 0 0 0))
   )
@@
   )
   (text "Only populate one\nDNP for FTDI" (at 77.47 64.77 90)
+    (effects (font (size 1.27 1.27)) (justify left bottom))
+  )
+  (label "USBB_D-" (at 104.14 76.2 0)
+    (effects (font (size 1.27 1.27)) (justify left bottom))
+  )
+  (label "FTDI_D+" (at 133.35 76.2 0)
+    (effects (font (size 1.27 1.27)) (justify left bottom))
+  )
+  (label "FTDI_RX_LED" (at 182.88 91.44 0)
+    (effects (font (size 1.27 1.27)) (justify left bottom))
+  )
+  (label "USBB_D+" (at 105.41 73.66 0)
+    (effects (font (size 1.27 1.27)) (justify left bottom))
+  )
+  (label "FTDI_TX_LED" (at 182.88 93.98 0)
+    (effects (font (size 1.27 1.27)) (justify left bottom))
+  )
+  (label "FTDI_VCC" (at 161.29 55.88 0)
+    (effects (font (size 1.27 1.27)) (justify left bottom))
+  )
+  (label "FTDI_D-" (at 133.35 73.66 0)
     (effects (font (size 1.27 1.27)) (justify left bottom))
   )
@@
     (pin "2")
   )
-  (symbol (lib_id "Interface_USB:FT231XS") (at 158.75 81.28 0) (unit 1)
-    (in_bom yes) (on_board yes) (fields_autoplaced)
-    (property "Reference" "U2" (id 0) (at 163.3094 57.15 0)
-      (effects (font (size 1.27 1.27)) (justify left))
-    )
-    (property "Value" "FT231XS" (id 1) (at 163.3094 59.69 0)
-      (effects (font (size 1.27 1.27)) (justify left))
-    )
-    (property "Footprint" "Package_SO:SSOP-20_3.9x8.7mm_P0.635mm" (id 2) (at 184.15 101.6 0)
+  (symbol (lib_id "Interface_USB:FT231XQ") (at 158.75 81.28 0) (unit 1)
+    (in_bom yes) (on_board yes)
+    (property "Reference" "U2" (id 0) (at 144.78 60.96 0)
+      (effects (font (size 1.27 1.27)) (justify left))
+    )
+    (property "Value" "FT231XQ" (id 1) (at 165.1 60.96 0)
+      (effects (font (size 1.27 1.27)) (justify left))
+    )
+    (property "Footprint" "Package_DFN_QFN:QFN-20-1EP_4x4mm_P0.5mm_EP2.5x2.5mm" (id 2) (at 193.04 101.6 0)
       (effects (font (size 1.27 1.27)) hide)
     )
@@
     (pin "2")
     (pin "20")
+    (pin "21")
     (pin "3")
     (pin "4")

Commit message: InterfaceBoard: Add STM32G0B1RET
Parts:
- added D? (x3): D_TVS, symbol Device:D_TVS
Connections:
- net GND: now also D?.1 (A1), D?.1 (A1), D?.1 (A1)
- net USBB_D+: now also D?.2 (A2)
- net USBB_D-: now also D?.2 (A2)
- net V_USB: now also D?.2 (A2)
- net USB_DM renamed USB_D-
- net USB_DP renamed USB_D+
Other:
- moved on the sheet: J2, R74

Commit message: InterfaceBoard: Make library paths relative
Parts:
- removed D? (x2): D_TVS, symbol Device:D_TVS
- added D5, D7: PE1605M1Q, Diode_SMD:D_0402_1005Metric, symbol Device:D_TVS
- D6: renamed from D?; value D_TVS -> PE1605M1Q; footprint (none) -> Diode_SMD:D_0402_1005Metric
Connections:
- net GND: now also D5.1 (A1), D7.1 (A1)
- net USBB_D+: now also D7.2 (A2)
- net V_USB: now also D5.2 (A2)
Changed lines of the file:
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@@
   (junction (at 63.5 71.12) (diameter 0) (color 0 0 0 0)
   )
-  (junction (at 63.5 96.52) (diameter 0) (color 0 0 0 0)
-  )
   (junction (at 198.12 55.88) (diameter 0) (color 0 0 0 0)
   )
@@
   (junction (at 149.86 39.37) (diameter 0) (color 0 0 0 0)
   )
+  (junction (at 63.5 102.87) (diameter 0) (color 0 0 0 0)
+  )
   (junction (at 90.17 68.58) (diameter 0) (color 0 0 0 0)
   )
@@
     (stroke (width 0) (type default) (color 0 0 0 0))
   )
-  (wire (pts (xy 59.69 96.52) (xy 63.5 96.52))
+  (wire (pts (xy 59.69 102.87) (xy 63.5 102.87))
     (stroke (width 0) (type default) (color 0 0 0 0))
   )
@@
     (stroke (width 0) (type default) (color 0 0 0 0))
   )
-  (wire (pts (xy 67.31 90.17) (xy 67.31 96.52))
+  (wire (pts (xy 67.31 90.17) (xy 67.31 102.87))
     (stroke (width 0) (type default) (color 0 0 0 0))
   )
@@
     (stroke (width 0) (type default) (color 0 0 0 0))
   )
-  (wire (pts (xy 63.5 90.17) (xy 63.5 96.52))
-    (stroke (width 0) (type default) (color 0 0 0 0))
-  )
   (polyline (pts (xy 209.55 114.3) (xy 209.55 31.75))
     (stroke (width 0) (type default) (color 0 0 0 0))
@@
     (stroke (width 0) (type default) (color 0 0 0 0))
   )
-  (wire (pts (xy 67.31 96.52) (xy 63.5 96.52))
+  (wire (pts (xy 67.31 102.87) (xy 63.5 102.87))
     (stroke (width 0) (type default) (color 0 0 0 0))
   )
@@
     (stroke (width 0) (type default) (color 0 0 0 0))
   )
+  (wire (pts (xy 63.5 90.17) (xy 63.5 102.87))
+    (stroke (width 0) (type default) (color 0 0 0 0))
+  )
   (polyline (pts (xy 86.36 64.77) (xy 77.47 64.77))
     (stroke (width 0) (type default) (color 0 0 0 0))
@@
     (stroke (width 0) (type default) (color 0 0 0 0))
   )
-  (wire (pts (xy 63.5 96.52) (xy 63.5 97.79))
+  (wire (pts (xy 63.5 102.87) (xy 63.5 104.14))
     (stroke (width 0) (type default) (color 0 0 0 0))
   )
@@
     (stroke (width 0) (type default) (color 0 0 0 0))
   )
-  (wire (pts (xy 59.69 90.17) (xy 59.69 96.52))
+  (wire (pts (xy 59.69 90.17) (xy 59.69 102.87))
     (stroke (width 0) (type default) (color 0 0 0 0))
   )
@@
     (pin "2")
   )
-  (symbol (lib_id "power:GND") (at 63.5 97.79 0) (unit 1)
-    (in_bom yes) (on_board yes)
-    (property "Reference" "#PWR?" (id 0) (at 63.5 104.14 0)
-      (effects (font (size 1.27 1.27)) hide)
-    )
-    (property "Value" "GND" (id 1) (at 63.5 101.6 0))
-    (property "Footprint" "" (id 2) (at 63.5 97.79 0)
-      (effects (font (size 1.27 1.27)) hide)
-    )
-    (property "Datasheet" "" (id 3) (at 63.5 97.79 0)
+  (symbol (lib_id "power:GND") (at 63.5 104.14 0) (unit 1)
+    (in_bom yes) (on_board yes)
+    (property "Reference" "#PWR0168" (id 0) (at 63.5 110.49 0)
+      (effects (font (size 1.27 1.27)) hide)
+    )
+    (property "Value" "GND" (id 1) (at 63.5 107.95 0))
+    (property "Footprint" "" (id 2) (at 63.5 104.14 0)
+      (effects (font (size 1.27 1.27)) hide)
+    )
+    (property "Datasheet" "" (id 3) (at 63.5 104.14 0)
       (effects (font (size 1.27 1.27)) hide)
     )
@@
     (pin "1")
   )
-  (symbol (lib_id "Device:D_TVS") (at 67.31 86.36 90) (unit 1)
-    (in_bom yes) (on_board yes)
-    (property "Reference" "D?" (id 0) (at 66.04 82.55 0)
-      (effects (font (size 1.27 1.27)) (justify left))
-    )
-    (property "Value" "D_TVS" (id 1) (at 66.04 90.17 0)
-      (effects (font (size 1.27 1.27)) (justify right))
-    )
-    (property "Footprint" "" (id 2) (at 67.31 86.36 0)
-      (effects (font (size 1.27 1.27)) hide)
-    )
-    (property "Datasheet" "~" (id 3) (at 67.31 86.36 0)
-      (effects (font (size 1.27 1.27)) hide)
-    )
-    (pin "1")
-    (pin "2")
-  )
   (symbol (lib_id "Device:C_Small") (at 97.79 82.55 0) (unit 1)
     (in_bom yes) (on_board yes)
@@
   (symbol (lib_id "Device:D_TVS") (at 63.5 86.36 90) (unit 1)
     (in_bom yes) (on_board yes)
-    (property "Reference" "D?" (id 0) (at 62.23 82.55 0)
-      (effects (font (size 1.27 1.27)) (justify left))
-    )
-    (property "Value" "D_TVS" (id 1) (at 62.23 90.17 0)
-      (effects (font (size 1.27 1.27)) (justify right))
-    )
-    (property "Footprint" "" (id 2) (at 63.5 86.36 0)
-      (effects (font (size 1.27 1.27)) hide)
-    )
-    (property "Datasheet" "~" (id 3) (at 63.5 86.36 0)
+    (property "Reference" "D6" (id 0) (at 62.23 82.55 0)
+      (effects (font (size 1.27 1.27)) (justify left))
+    )
+    (property "Value" "PE1605M1Q" (id 1) (at 62.23 90.17 0)
+      (effects (font (size 1.27 1.27)) (justify right))
+    )
+    (property "Footprint" "Diode_SMD:D_0402_1005Metric" (id 2) (at 63.5 86.36 0)
+      (effects (font (size 1.27 1.27)) hide)
+    )
+    (property "Datasheet" "https://www.panjit.com.tw/upload/datasheet/PE1605M1Q.pdf" (id 3) (at 63.5 86.36 0)
       (effects (font (size 1.27 1.27)) hide)
     )
@@
     (pin "2")
   )
+  (symbol (lib_id "Device:D_TVS") (at 59.69 86.36 90) (unit 1)
+    (in_bom yes) (on_board yes)
+    (property "Reference" "D5" (id 0) (at 58.42 82.55 0)
+      (effects (font (size 1.27 1.27)) (justify left))
+    )
+    (property "Value" "PE1605M1Q" (id 1) (at 58.42 90.17 0)
+      (effects (font (size 1.27 1.27)) (justify right))
+    )
+    (property "Footprint" "Diode_SMD:D_0402_1005Metric" (id 2) (at 59.69 86.36 0)
+      (effects (font (size 1.27 1.27)) hide)
+    )
+    (property "Datasheet" "https://www.panjit.com.tw/upload/datasheet/PE1605M1Q.pdf" (id 3) (at 59.69 86.36 0)
+      (effects (font (size 1.27 1.27)) hide)
+    )
+    (pin "1")
+    (pin "2")
+  )
   (symbol (lib_id "Device:LED_Small") (at 201.93 80.01 90) (unit 1)
     (in_bom yes) (on_board yes)
@@
     )
     (property "Datasheet" "~" (id 3) (at 50.8 88.9 0)
-      (effects (font (size 1.27 1.27)) hide)
-    )
-    (pin "1")
-    (pin "2")
-  )
-  (symbol (lib_id "Device:D_TVS") (at 59.69 86.36 90) (unit 1)
-    (in_bom yes) (on_board yes)
-    (property "Reference" "D?" (id 0) (at 58.42 82.55 0)
-      (effects (font (size 1.27 1.27)) (justify left))
-    )
-    (property "Value" "D_TVS" (id 1) (at 58.42 90.17 0)
-      (effects (font (size 1.27 1.27)) (justify right))
-    )
-    (property "Footprint" "" (id 2) (at 59.69 86.36 0)
-      (effects (font (size 1.27 1.27)) hide)
-    )
-    (property "Datasheet" "~" (id 3) (at 59.69 86.36 0)
       (effects (font (size 1.27 1.27)) hide)
     )
@@
     (pin "1")
   )
+  (symbol (lib_id "Device:D_TVS") (at 67.31 86.36 90) (unit 1)
+    (in_bom yes) (on_board yes)
+    (property "Reference" "D7" (id 0) (at 66.04 82.55 0)
+      (effects (font (size 1.27 1.27)) (justify left))
+    )
+    (property "Value" "PE1605M1Q" (id 1) (at 66.04 90.17 0)
+      (effects (font (size 1.27 1.27)) (justify right))
+    )
+    (property "Footprint" "Diode_SMD:D_0402_1005Metric" (id 2) (at 67.31 86.36 0)
+      (effects (font (size 1.27 1.27)) hide)
+    )
+    (property "Datasheet" "https://www.panjit.com.tw/upload/datasheet/PE1605M1Q.pdf" (id 3) (at 67.31 86.36 0)
+      (effects (font (size 1.27 1.27)) hide)
+    )
+    (pin "1")
+    (pin "2")
+  )
   (symbol (lib_id "Device:R_Small") (at 120.65 76.2 90) (unit 1)

Commit message: InterfaceBoard: Add 3.3 V regulater, test points.
Parts:
- U2: DigiKey (none) -> https://www.digikey.com/en/products/detail/ftdi-future-tech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
Changed lines of the file:
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@@
+      (effects (font (size 1.27 1.27)) hide)
+    )
+    (property "DigiKey" "https://www.digikey.com/en/products/detail/ftdi-future-technology-devices-international-ltd/FT231XQ-T/3749470" (id 4) (at 158.75 81.28 0)
       (effects (font (size 1.27 1.27)) hide)
     )

Commit message: InterfaceBoard: Place and route buttons and LEDs.
Parts:
- added Q4: BC856W, Package_TO_SOT_SMD:SOT-323_SC-70, symbol Transistor_BJT:BC856W
- added R86: 10k, Resistor_SMD:R_0603_1608Metric, symbol Device:R_Small
- added R87: 180k, Resistor_SMD:R_0603_1608Metric, symbol Device:R_Small
- added R88: 0, Resistor_SMD:R_0603_1608Metric, symbol Device:R_Small
Connections:
- net USB_PULLUP: now also R86.1, R88.2; no longer R75.2, R76.2
- new net: Q4.1 (B), R86.2, R87.1
- new net: Q4.3 (C), R75.2, R76.2, R88.1
- new net +3V3: Q4.2 (E), R87.2
Other:
- note added: "Populate either 0-ohm jumper, or PNP transistor network."

Commit message: InterfaceBoard: Route MCU USB
Parts:
- added R93, R94: 0, Resistor_SMD:R_0603_1608Metric, symbol Device:R_Small
- R17, R18, R19, R20: value 27R -> 27
Connections:
- net USBB_D+: now also R93.1; no longer R17.1
- net USBB_D-: now also R94.1; no longer R18.1
- new net MCU_USBB_D+: R17.1, R93.2
- new net MCU_USBB_D-: R18.1, R94.2
Other:
- moved on the sheet: R17, R18
Changed lines of the file:
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@@
     (stroke (width 0) (type default) (color 0 0 0 0))
   )
-  (polyline (pts (xy 107.95 40.64) (xy 107.95 71.12))
+  (polyline (pts (xy 107.95 25.4) (xy 107.95 67.31))
     (stroke (width 0) (type default) (color 0 0 0 0))
   )
@@
     (stroke (width 0) (type default) (color 0 0 0 0))
   )
-  (wire (pts (xy 104.14 55.88) (xy 104.14 60.96))
+  (wire (pts (xy 104.14 40.64) (xy 104.14 45.72))
     (stroke (width 0) (type default) (color 0 0 0 0))
   )
@@
     (stroke (width 0) (type default) (color 0 0 0 0))
   )
-  (polyline (pts (xy 107.95 71.12) (xy 95.25 71.12))
+  (polyline (pts (xy 107.95 67.31) (xy 95.25 67.31))
+    (stroke (width 0) (type default) (color 0 0 0 0))
+  )
+  (wire (pts (xy 104.14 63.5) (xy 104.14 76.2))
     (stroke (width 0) (type default) (color 0 0 0 0))
   )
@@
     (stroke (width 0) (type default) (color 0 0 0 0))
   )
-  (wire (pts (xy 104.14 66.04) (xy 104.14 76.2))
+  (wire (pts (xy 104.14 50.8) (xy 104.14 58.42))
     (stroke (width 0) (type default) (color 0 0 0 0))
   )
@@
     (stroke (width 0) (type default) (color 0 0 0 0))
   )
-  (polyline (pts (xy 95.25 71.12) (xy 95.25 40.64))
+  (polyline (pts (xy 95.25 67.31) (xy 95.25 25.4))
     (stroke (width 0) (type default) (color 0 0 0 0))
   )
@@
     (stroke (width 0) (type default) (color 0 0 0 0))
   )
-  (wire (pts (xy 101.6 66.04) (xy 101.6 73.66))
+  (wire (pts (xy 101.6 50.8) (xy 101.6 58.42))
     (stroke (width 0) (type default) (color 0 0 0 0))
   )
@@
     (stroke (width 0) (type default) (color 0 0 0 0))
   )
-  (polyline (pts (xy 95.25 40.64) (xy 107.95 40.64))
+  (polyline (pts (xy 95.25 25.4) (xy 107.95 25.4))
     (stroke (width 0) (type default) (color 0 0 0 0))
   )
@@
     (stroke (width 0) (type default) (color 0 0 0 0))
   )
+  (wire (pts (xy 101.6 63.5) (xy 101.6 73.66))
+    (stroke (width 0) (type default) (color 0 0 0 0))
+  )
   (wire (pts (xy 59.69 90.17) (xy 59.69 102.87))
     (stroke (width 0) (type default) (color 0 0 0 0))
@@
     (stroke (width 0) (type default) (color 0 0 0 0))
   )
-  (wire (pts (xy 101.6 55.88) (xy 101.6 60.96))
+  (wire (pts (xy 101.6 40.64) (xy 101.6 45.72))
     (stroke (width 0) (type default) (color 0 0 0 0))
   )
@@
     (stroke (width 0) (type default) (color 0 0 0 0))
   )
-  (text "Option A\nMCU USB" (at 96.52 45.72 0)
+  (text "Option A\nMCU USB" (at 96.52 30.48 0)
     (effects (font (size 1.27 1.27)) (justify left bottom))
   )
@@
     (effects (font (size 1.27 1.27)) (justify left bottom))
   )
+  (label "MCU_USBB_D-" (at 104.14 54.61 0)
+    (effects (font (size 1.27 1.27)) (justify left bottom))
+  )
+  (label "MCU_USBB_D+" (at 101.6 57.15 0)
+    (effects (font (size 1.27 1.27)) (justify left bottom))
+  )
   (label "FTDI_TX_LED" (at 182.88 93.98 0)
     (effects (font (size 1.27 1.27)) (justify left bottom))
@@
     (effects (font (size 1.27 1.27)) (justify left))
   )
-  (hierarchical_label "USB_D-" (shape bidirectional) (at 104.14 55.88 90)
+  (hierarchical_label "USB_D-" (shape bidirectional) (at 104.14 40.64 90)
     (effects (font (size 1.27 1.27)) (justify left))
   )
@@
     (effects (font (size 1.27 1.27)) (justify left))
   )
-  (hierarchical_label "USB_D+" (shape bidirectional) (at 101.6 55.88 90)
+  (hierarchical_label "USB_D+" (shape bidirectional) (at 101.6 40.64 90)
     (effects (font (size 1.27 1.27)) (justify left))
   )
@@
       (effects (font (size 1.27 1.27)) (justify left))
     )
-    (property "Value" "27R" (id 1) (at 123.19 71.12 90)
+    (property "Value" "27" (id 1) (at 123.19 71.12 90)
       (effects (font (size 1.27 1.27)) (justify right))
     )
@@
     (pin "1")
   )
-  (symbol (lib_id "Device:R_Small") (at 101.6 63.5 180) (unit 1)
-    (in_bom yes) (on_board yes)
-    (property "Reference" "R17" (id 0) (at 100.33 66.04 90)
-      (effects (font (size 1.27 1.27)) (justify left))
-    )
-    (property "Value" "27R" (id 1) (at 100.33 60.96 90)
-      (effects (font (size 1.27 1.27)) (justify right))
-    )
-    (property "Footprint" "Resistor_SMD:R_0603_1608Metric" (id 2) (at 101.6 63.5 0)
-      (effects (font (size 1.27 1.27)) hide)
-    )
-    (property "Datasheet" "~" (id 3) (at 101.6 63.5 0)
+  (symbol (lib_id "Device:R_Small") (at 101.6 48.26 180) (unit 1)
+    (in_bom yes) (on_board yes)
+    (property "Reference" "R17" (id 0) (at 100.33 50.8 90)
+      (effects (font (size 1.27 1.27)) (justify left))
+    )
+    (property "Value" "27" (id 1) (at 100.33 45.72 90)
+      (effects (font (size 1.27 1.27)) (justify right))
+    )
+    (property "Footprint" "Resistor_SMD:R_0603_1608Metric" (id 2) (at 101.6 48.26 0)
+      (effects (font (size 1.27 1.27)) hide)
+    )
+    (property "Datasheet" "~" (id 3) (at 101.6 48.26 0)
       (effects (font (size 1.27 1.27)) hide)
     )
@@
       (effects (font (size 1.27 1.27)) (justify left))
     )
-    (property "Value" "27R" (id 1) (at 123.19 74.93 90)
+    (property "Value" "27" (id 1) (at 123.19 74.93 90)
       (effects (font (size 1.27 1.27)) (justify right))
     )
@@
     (pin "2")
   )
-  (symbol (lib_id "Device:R_Small") (at 104.14 63.5 180) (unit 1)
-    (in_bom yes) (on_board yes)
-    (property "Reference" "R18" (id 0) (at 102.87 66.04 90)
-      (effects (font (size 1.27 1.27)) (justify left))
-    )
-    (property "Value" "27R" (id 1) (at 102.87 60.96 90)
-      (effects (font (size 1.27 1.27)) (justify right))
-    )
-    (property "Footprint" "Resistor_SMD:R_0603_1608Metric" (id 2) (at 104.14 63.5 0)
-      (effects (font (size 1.27 1.27)) hide)
-    )
-    (property "Datasheet" "~" (id 3) (at 104.14 63.5 0)
+  (symbol (lib_id "Device:R_Small") (at 104.14 48.26 180) (unit 1)
+    (in_bom yes) (on_board yes)
+    (property "Reference" "R18" (id 0) (at 102.87 50.8 90)
+      (effects (font (size 1.27 1.27)) (justify left))
+    )
+    (property "Value" "27" (id 1) (at 102.87 45.72 90)
+      (effects (font (size 1.27 1.27)) (justify right))
+    )
+    (property "Footprint" "Resistor_SMD:R_0603_1608Metric" (id 2) (at 104.14 48.26 0)
+      (effects (font (size 1.27 1.27)) hide)
+    )
+    (property "Datasheet" "~" (id 3) (at 104.14 48.26 0)
+      (effects (font (size 1.27 1.27)) hide)
+    )
+    (pin "1")
+    (pin "2")
+  )
+  (symbol (lib_id "Device:R_Small") (at 101.6 60.96 180) (unit 1)
+    (in_bom yes) (on_board yes)
+    (property "Reference" "R93" (id 0) (at 100.33 63.5 90)
+      (effects (font (size 1.27 1.27)) (justify left))
+    )
+    (property "Value" "0" (id 1) (at 100.33 58.42 90)
+      (effects (font (size 1.27 1.27)) (justify right))
+    )
+    (property "Footprint" "Resistor_SMD:R_0603_1608Metric" (id 2) (at 101.6 60.96 0)
+      (effects (font (size 1.27 1.27)) hide)
+    )
+    (property "Datasheet" "~" (id 3) (at 101.6 60.96 0)
       (effects (font (size 1.27 1.27)) hide)
     )
@@
       (effects (font (size 1.27 1.27)) hide)
     )
+    (pin "1")
+    (pin "2")
+  )
+  (symbol (lib_id "Device:R_Small") (at 104.14 60.96 180) (unit 1)
+    (in_bom yes) (on_board yes)
+    (property "Reference" "R94" (id 0) (at 102.87 63.5 90)
+      (effects (font (size 1.27 1.27)) (justify left))
+    )
+    (property "Value" "0" (id 1) (at 102.87 58.42 90)
+      (effects (font (size 1.27 1.27)) (justify right))
+    )
+    (property "Footprint" "Resistor_SMD:R_0603_1608Metric" (id 2) (at 104.14 60.96 0)
+      (effects (font (size 1.27 1.27)) hide)
+    )
+    (property "Datasheet" "~" (id 3) (at 104.14 60.96 0)
+      (effects (font (size 1.27 1.27)) hide)
+    )
