File: InterfaceBoard/USB.kicad_sch (KiCad schematic)
At the start: 28 parts, among them J2 USB_B, Q4 BC856W, U2 FT231XQ

Commit message: InterfaceBoard: Rev 1.0
Parts:
- renumbered C21 to C34, C22 to C35, C20 to C36, C19 to C37, C17 to C38, C18 to C39, D5 to D10, D7 to D11, D6 to D12, D3 to D4, D4 to D9, J2 to J7, R17 to R37, R18 to R40, R21 to R57, R20 to R64, R19 to R67, R93 to R70, R94 to R71, R22 to R76, R88 to R77, R87 to R78, R86 to R79, R74 to R87, R76 to R88, R75 to R89, U2 to U4
Other:
- company: (none) -> Peter Farley
- title: (none) -> Kiethley 615 Interface Board
Changed lines of the file:
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@@
 (kicad_sch (version 20211123) (generator eeschema)
   (paper "A4")
+  (title_block
+    (title "Kiethley 615 Interface Board")
+    (date "2023-03-04")
+    (rev "1.0")
+    (company "Peter Farley")
+    (comment 1 "Rev 1.0: Initial revision")
+  )
   (junction (at 82.55 46.99) (diameter 0) (color 0 0 0 0)
   )
@@
   (symbol (lib_id "lib_symbols:UJ2-BH-W1-TH") (at 39.37 73.66 0) (unit 1)
     (in_bom yes) (on_board yes) (fields_autoplaced)
-    (property "Reference" "J2" (id 0) (at 39.37 60.96 0))
+    (property "Reference" "J7" (id 0) (at 39.37 60.96 0))
     (property "Value" "USB_B" (id 1) (at 39.37 63.5 0))
     (property "Footprint" "lib:CUI_UJ2-BH-W1-TH" (id 2) (at 40.64 63.5 0)
@@
   (symbol (lib_id "Device:R_Small") (at 201.93 68.58 180) (unit 1)
     (in_bom yes) (on_board yes)
-    (property "Reference" "R22" (id 0) (at 200.66 66.04 90)
+    (property "Reference" "R76" (id 0) (at 200.66 66.04 90)
       (effects (font (size 1.27 1.27)) (justify right))
     )
@@
   (symbol (lib_id "Device:C_Small") (at 93.98 82.55 0) (unit 1)
     (in_bom yes) (on_board yes)
-    (property "Reference" "C18" (id 0) (at 92.71 81.28 90)
+    (property "Reference" "C39" (id 0) (at 92.71 81.28 90)
       (effects (font (size 1.27 1.27)) (justify left))
     )
@@
   (symbol (lib_id "Device:R_Small") (at 69.85 27.94 0) (mirror x) (unit 1)
     (in_bom yes) (on_board yes)
-    (property "Reference" "R87" (id 0) (at 71.12 30.48 90)
+    (property "Reference" "R78" (id 0) (at 71.12 30.48 90)
       (effects (font (size 1.27 1.27)) (justify left))
     )
@@
   (symbol (lib_id "Device:LED_Small") (at 198.12 80.01 90) (unit 1)
     (in_bom yes) (on_board yes)
-    (property "Reference" "D3" (id 0) (at 196.85 76.2 0)
+    (property "Reference" "D4" (id 0) (at 196.85 76.2 0)
       (effects (font (size 1.27 1.27)) (justify right))
     )
@@
   (symbol (lib_id "Device:R_Small") (at 198.12 68.58 180) (unit 1)
     (in_bom yes) (on_board yes)
-    (property "Reference" "R21" (id 0) (at 196.85 66.04 90)
+    (property "Reference" "R57" (id 0) (at 196.85 66.04 90)
       (effects (font (size 1.27 1.27)) (justify right))
     )
@@
   (symbol (lib_id "Device:C_Small") (at 97.79 82.55 0) (unit 1)
     (in_bom yes) (on_board yes)
-    (property "Reference" "C19" (id 0) (at 96.52 81.28 90)
+    (property "Reference" "C37" (id 0) (at 96.52 81.28 90)
       (effects (font (size 1.27 1.27)) (justify left))
     )
@@
   (symbol (lib_id "Device:C_Small") (at 90.17 82.55 0) (unit 1)
     (in_bom yes) (on_board yes)
-    (property "Reference" "C17" (id 0) (at 88.9 81.28 90)
+    (property "Reference" "C38" (id 0) (at 88.9 81.28 90)
       (effects (font (size 1.27 1.27)) (justify left))
     )
@@
   (symbol (lib_id "Device:R_Small") (at 81.28 57.15 180) (unit 1)
     (in_bom yes) (on_board yes)
-    (property "Reference" "R75" (id 0) (at 80.01 59.69 90)
+    (property "Reference" "R89" (id 0) (at 80.01 59.69 90)
       (effects (font (size 1.27 1.27)) (justify left))
     )
@@
   (symbol (lib_id "Device:R_Small") (at 66.04 35.56 90) (mirror x) (unit 1)
     (in_bom yes) (on_board yes)
-    (property "Reference" "R86" (id 0) (at 63.5 36.83 90)
+    (property "Reference" "R79" (id 0) (at 63.5 36.83 90)
       (effects (font (size 1.27 1.27)) (justify left))
     )
@@
   (symbol (lib_id "Device:D_TVS") (at 63.5 86.36 90) (unit 1)
     (in_bom yes) (on_board yes)
-    (property "Reference" "D6" (id 0) (at 62.23 82.55 0)
+    (property "Reference" "D12" (id 0) (at 62.23 82.55 0)
       (effects (font (size 1.27 1.27)) (justify left))
     )
@@
   (symbol (lib_id "Device:R_Small") (at 83.82 57.15 180) (unit 1)
     (in_bom yes) (on_board yes)
-    (property "Reference" "R76" (id 0) (at 82.55 59.69 90)
+    (property "Reference" "R88" (id 0) (at 82.55 59.69 90)
       (effects (font (size 1.27 1.27)) (justify left))
     )
@@
   (symbol (lib_id "Device:R_Small") (at 120.65 72.39 90) (unit 1)
     (in_bom yes) (on_board yes)
-    (property "Reference" "R19" (id 0) (at 118.11 71.12 90)
+    (property "Reference" "R67" (id 0) (at 118.11 71.12 90)
       (effects (font (size 1.27 1.27)) (justify left))
     )
@@
   (symbol (lib_id "Device:R_Small") (at 101.6 48.26 180) (unit 1)
     (in_bom yes) (on_board yes)
-    (property "Reference" "R17" (id 0) (at 100.33 50.8 90)
+    (property "Reference" "R37" (id 0) (at 100.33 50.8 90)
       (effects (font (size 1.27 1.27)) (justify left))
     )
@@
   (symbol (lib_id "Device:C_Small") (at 146.05 44.45 0) (unit 1)
     (in_bom yes) (on_board yes)
-    (property "Reference" "C21" (id 0) (at 144.78 43.18 90)
+    (property "Reference" "C34" (id 0) (at 144.78 43.18 90)
       (effects (font (size 1.27 1.27)) (justify left))
     )
@@
   (symbol (lib_id "Device:D_TVS") (at 59.69 86.36 90) (unit 1)
     (in_bom yes) (on_board yes)
-    (property "Reference" "D5" (id 0) (at 58.42 82.55 0)
+    (property "Reference" "D10" (id 0) (at 58.42 82.55 0)
       (effects (font (size 1.27 1.27)) (justify left))
     )
@@
   (symbol (lib_id "Device:LED_Small") (at 201.93 80.01 90) (unit 1)
     (in_bom yes) (on_board yes)
-    (property "Reference" "D4" (id 0) (at 200.66 76.2 0)
+    (property "Reference" "D9" (id 0) (at 200.66 76.2 0)
       (effects (font (size 1.27 1.27)) (justify right))
     )
@@
   (symbol (lib_id "Device:R_Small") (at 50.8 88.9 180) (unit 1)
     (in_bom yes) (on_board yes)
-    (property "Reference" "R74" (id 0) (at 49.53 91.44 90)
+    (property "Reference" "R87" (id 0) (at 49.53 91.44 90)
       (effects (font (size 1.27 1.27)) (justify left))
     )
@@
   (symbol (lib_id "Device:D_TVS") (at 67.31 86.36 90) (unit 1)
     (in_bom yes) (on_board yes)
-    (property "Reference" "D7" (id 0) (at 66.04 82.55 0)
+    (property "Reference" "D11" (id 0) (at 66.04 82.55 0)
       (effects (font (size 1.27 1.27)) (justify left))
     )
@@
   (symbol (lib_id "Device:R_Small") (at 120.65 76.2 90) (unit 1)
     (in_bom yes) (on_board yes)
-    (property "Reference" "R20" (id 0) (at 118.11 74.93 90)
+    (property "Reference" "R64" (id 0) (at 118.11 74.93 90)
       (effects (font (size 1.27 1.27)) (justify left))
     )
@@
   (symbol (lib_id "Device:R_Small") (at 104.14 48.26 180) (unit 1)
     (in_bom yes) (on_board yes)
-    (property "Reference" "R18" (id 0) (at 102.87 50.8 90)
+    (property "Reference" "R40" (id 0) (at 102.87 50.8 90)
       (effects (font (size 1.27 1.27)) (justify left))
     )
@@
   (symbol (lib_id "Device:R_Small") (at 101.6 60.96 180) (unit 1)
     (in_bom yes) (on_board yes)
-    (property "Reference" "R93" (id 0) (at 100.33 63.5 90)
+    (property "Reference" "R70" (id 0) (at 100.33 63.5 90)
       (effects (font (size 1.27 1.27)) (justify left))
     )
@@
   (symbol (lib_id "Device:C_Small") (at 149.86 44.45 0) (unit 1)
     (in_bom yes) (on_board yes)
-    (property "Reference" "C22" (id 0) (at 148.59 43.18 90)
+    (property "Reference" "C35" (id 0) (at 148.59 43.18 90)
       (effects (font (size 1.27 1.27)) (justify left))
     )
@@
   (symbol (lib_id "Device:R_Small") (at 104.14 60.96 180) (unit 1)
     (in_bom yes) (on_board yes)
-    (property "Reference" "R94" (id 0) (at 102.87 63.5 90)
+    (property "Reference" "R71" (id 0) (at 102.87 63.5 90)
       (effects (font (size 1.27 1.27)) (justify left))
     )
@@
   (symbol (lib_id "Device:R_Small") (at 85.09 35.56 180) (unit 1)
     (in_bom yes) (on_board yes)
-    (property "Reference" "R88" (id 0) (at 83.82 38.1 90)
+    (property "Reference" "R77" (id 0) (at 83.82 38.1 90)
       (effects (font (size 1.27 1.27)) (justify left))
     )
@@
   (symbol (lib_id "Interface_USB:FT231XQ") (at 158.75 81.28 0) (unit 1)
     (in_bom yes) (on_board yes)
-    (property "Reference" "U2" (id 0) (at 144.78 60.96 0)
+    (property "Reference" "U4" (id 0) (at 144.78 60.96 0)
       (effects (font (size 1.27 1.27)) (justify left))
     )
@@
   (symbol (lib_id "Device:C_Small") (at 135.89 59.69 0) (unit 1)
     (in_bom yes) (on_board yes)
-    (property "Reference" "C20" (id 0) (at 134.62 58.42 90)
-      (effects (font (size 1.27 1.27)) (justify left))
-    )
+    (property "Reference" "C36" (id 0) (at 134.62 58.42 90)
+      (effects (font (size 1.27 1.27)) (justify left))
+    )

Commit message: InterfaceBoard: Add BOM
Parts:
- C34, C35: DigiKey (none) -> https://www.digikey.com/en/products/detail/samsung-electro-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
- C36, C37, C38, C39, R57, R70, R71, R76, R77, R87, R88, R89: DigiKey (none) -> https://www.digikey.com/en/products/detail/walsin-technolog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
- D10, D11, D12: DigiKey (none) -> https://www.digikey.com/en/products/detail/panjit-internati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
- D4, D9: DigiKey (none) -> https://www.digikey.com/en/products/detail/harvatek-corpora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
- J7: DigiKey (none) -> https://www.digikey.com/en/products/detail/cui-devices/UJ2-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
- R37, R40, R64, R67: DigiKey (none) -> https://www.digikey.com/en/products/detail/stackpole-electr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
- R78, R79: DigiKey (none) -> https://www.digikey.com/en/products/detail/yageo/RC0603FR-1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
Changed lines of the file:
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@@
       (effects (font (size 1.27 1.27)) (justify bottom) hide)
     )
-    (property "Datasheet" " ~" (id 3) (at 39.37 73.66 0)
+    (property "Datasheet" "https://www.cuidevices.com/product/resource/uj2-bh-th.pdf" (id 3) (at 39.37 73.66 0)
       (effects (font (size 1.27 1.27)) hide)
     )
@@
     (property "STANDARD" "MANUFACTURER RECOMENDATION" (id 6) (at 39.37 88.9 0)
       (effects (font (size 1.27 1.27)) (justify bottom) hide)
+    )
+    (property "DigiKey" "https://www.digikey.com/en/products/detail/cui-devices/UJ2-BH-W1-TH/6188082" (id 7) (at 39.37 73.66 0)
+      (effects (font (size 1.27 1.27)) hide)
     )
     (pin "1")
@@
       (effects (font (size 1.27 1.27)) hide)
     )
+    (property "DigiKey" "https://www.digikey.com/en/products/detail/walsin-technology-corporation/WR06X102-JTL/13241138" (id 4) (at 201.93 68.58 0)
+      (effects (font (size 1.27 1.27)) hide)
+    )
     (pin "1")
     (pin "2")
@@
     )
     (property "Datasheet" "~" (id 3) (at 93.98 82.55 0)
+      (effects (font (size 1.27 1.27)) hide)
+    )
+    (property "DigiKey" "https://www.digikey.com/en/products/detail/walsin-technology-corporation/0603N470J500CT/9355025" (id 4) (at 93.98 82.55 0)
       (effects (font (size 1.27 1.27)) hide)
     )
@@
       (effects (font (size 1.27 1.27)) hide)
     )
+    (property "DigiKey" "https://www.digikey.com/en/products/detail/yageo/RC0603FR-10180KL/14008354" (id 4) (at 69.85 27.94 0)
+      (effects (font (size 1.27 1.27)) hide)
+    )
     (pin "1")
     (pin "2")
@@
       (effects (font (size 1.27 1.27)) hide)
     )
+    (property "DigiKey" "https://www.digikey.com/en/products/detail/harvatek-corporation/B1911USD-20D000114U1930/15519991" (id 4) (at 198.12 80.01 0)
+      (effects (font (size 1.27 1.27)) hide)
+    )
     (pin "1")
     (pin "2")
@@
     )
     (property "Datasheet" "~" (id 3) (at 198.12 68.58 0)
+      (effects (font (size 1.27 1.27)) hide)
+    )
+    (property "DigiKey" "https://www.digikey.com/en/products/detail/walsin-technology-corporation/WR06X102-JTL/13241138" (id 4) (at 198.12 68.58 0)
       (effects (font (size 1.27 1.27)) hide)
     )
@@
       (effects (font (size 1.27 1.27)) hide)
     )
+    (property "DigiKey" "https://www.digikey.com/en/products/detail/walsin-technology-corporation/0603B103K500CT/9354883" (id 4) (at 97.79 82.55 0)
+      (effects (font (size 1.27 1.27)) hide)
+    )
     (pin "1")
     (pin "2")
@@
       (effects (font (size 1.27 1.27)) hide)
     )
+    (property "DigiKey" "https://www.digikey.com/en/products/detail/walsin-technology-corporation/0603N470J500CT/9355025" (id 4) (at 90.17 82.55 0)
+      (effects (font (size 1.27 1.27)) hide)
+    )
     (pin "1")
     (pin "2")
@@
       (effects (font (size 1.27 1.27)) hide)
     )
+    (property "DigiKey" "https://www.digikey.com/en/products/detail/walsin-technology-corporation/WR06X1501FTL/13239261" (id 4) (at 81.28 57.15 0)
+      (effects (font (size 1.27 1.27)) hide)
+    )
     (pin "1")
     (pin "2")
@@
       (effects (font (size 1.27 1.27)) hide)
     )
+    (property "DigiKey" "https://www.digikey.com/en/products/detail/yageo/RC0603FR-1010KL/12756395" (id 4) (at 66.04 35.56 0)
+      (effects (font (size 1.27 1.27)) hide)
+    )
     (pin "1")
     (pin "2")
@@
     )
     (property "Datasheet" "https://www.panjit.com.tw/upload/datasheet/PE1605M1Q.pdf" (id 3) (at 63.5 86.36 0)
+      (effects (font (size 1.27 1.27)) hide)
+    )
+    (property "DigiKey" "https://www.digikey.com/en/products/detail/panjit-international-inc/PE1605M1Q-R1-00001/15798503" (id 4) (at 63.5 86.36 0)
       (effects (font (size 1.27 1.27)) hide)
     )
@@
       (effects (font (size 1.27 1.27)) hide)
     )
+    (property "DigiKey" "https://www.digikey.com/en/products/detail/walsin-technology-corporation/WR06X1501FTL/13239261" (id 4) (at 83.82 57.15 0)
+      (effects (font (size 1.27 1.27)) hide)
+    )
     (pin "1")
     (pin "2")
@@
     )
     (property "Datasheet" "~" (id 3) (at 120.65 72.39 0)
+      (effects (font (size 1.27 1.27)) hide)
+    )
+    (property "DigiKey" "https://www.digikey.com/en/products/detail/stackpole-electronics-inc/RMCF0603FT27R0/1760818" (id 4) (at 120.65 72.39 0)
       (effects (font (size 1.27 1.27)) hide)
     )
@@
       (effects (font (size 1.27 1.27)) hide)
     )
+    (property "DigiKey" "https://www.digikey.com/en/products/detail/stackpole-electronics-inc/RMCF0603FT27R0/1760818" (id 4) (at 101.6 48.26 0)
+      (effects (font (size 1.27 1.27)) hide)
+    )
     (pin "1")
     (pin "2")
@@
       (effects (font (size 1.27 1.27)) hide)
     )
+    (property "DigiKey" "https://www.digikey.com/en/products/detail/samsung-electro-mechanics/CL10B104KB8NNWC/3887593" (id 4) (at 146.05 44.45 0)
+      (effects (font (size 1.27 1.27)) hide)
+    )
     (pin "1")
     (pin "2")
@@
       (effects (font (size 1.27 1.27)) hide)
     )
+    (property "DigiKey" "https://www.digikey.com/en/products/detail/panjit-international-inc/PE1605M1Q-R1-00001/15798503" (id 4) (at 59.69 86.36 0)
+      (effects (font (size 1.27 1.27)) hide)
+    )
     (pin "1")
     (pin "2")
@@
     )
     (property "Datasheet" "~" (id 3) (at 201.93 80.01 90)
+      (effects (font (size 1.27 1.27)) hide)
+    )
+    (property "DigiKey" "https://www.digikey.com/en/products/detail/harvatek-corporation/B1911USD-20D000114U1930/15519991" (id 4) (at 201.93 80.01 0)
       (effects (font (size 1.27 1.27)) hide)
     )
@@
       (effects (font (size 1.27 1.27)) hide)
     )
+    (property "DigiKey" "https://www.digikey.com/en/products/detail/walsin-technology-corporation/WR06X000-PTL/5978108" (id 4) (at 50.8 88.9 0)
+      (effects (font (size 1.27 1.27)) hide)
+    )
     (pin "1")
     (pin "2")
@@
       (effects (font (size 1.27 1.27)) hide)
     )
+    (property "DigiKey" "https://www.digikey.com/en/products/detail/panjit-international-inc/PE1605M1Q-R1-00001/15798503" (id 4) (at 67.31 86.36 0)
+      (effects (font (size 1.27 1.27)) hide)
+    )
     (pin "1")
     (pin "2")
@@
       (effects (font (size 1.27 1.27)) hide)
     )
+    (property "DigiKey" "https://www.digikey.com/en/products/detail/stackpole-electronics-inc/RMCF0603FT27R0/1760818" (id 4) (at 120.65 76.2 0)
+      (effects (font (size 1.27 1.27)) hide)
+    )
     (pin "1")
     (pin "2")
@@
       (effects (font (size 1.27 1.27)) hide)
     )
+    (property "DigiKey" "https://www.digikey.com/en/products/detail/stackpole-electronics-inc/RMCF0603FT27R0/1760818" (id 4) (at 104.14 48.26 0)
+      (effects (font (size 1.27 1.27)) hide)
+    )
     (pin "1")
     (pin "2")
@@
       (effects (font (size 1.27 1.27)) hide)
     )
+    (property "DigiKey" "https://www.digikey.com/en/products/detail/walsin-technology-corporation/WR06X000-PTL/5978108" (id 4) (at 101.6 60.96 0)
+      (effects (font (size 1.27 1.27)) hide)
+    )
     (pin "1")
     (pin "2")
@@
       (effects (font (size 1.27 1.27)) hide)
     )
+    (property "DigiKey" "https://www.digikey.com/en/products/detail/samsung-electro-mechanics/CL10A475KQ8NNNC/3886703" (id 4) (at 149.86 44.45 0)
+      (effects (font (size 1.27 1.27)) hide)
+    )
     (pin "1")
     (pin "2")
@@
       (effects (font (size 1.27 1.27)) hide)
     )
+    (property "DigiKey" "https://www.digikey.com/en/products/detail/walsin-technology-corporation/WR06X000-PTL/5978108" (id 4) (at 104.14 60.96 0)
+      (effects (font (size 1.27 1.27)) hide)
+    )
     (pin "1")
     (pin "2")
@@
     )
     (property "Datasheet" "~" (id 3) (at 85.09 35.56 0)
+      (effects (font (size 1.27 1.27)) hide)
+    )
+    (property "DigiKey" "https://www.digikey.com/en/products/detail/walsin-technology-corporation/WR06X000-PTL/5978108" (id 4) (at 85.09 35.56 0)
       (effects (font (size 1.27 1.27)) hide)
     )
@@
       (effects (font (size 1.27 1.27)) hide)
     )
+    (property "DigiKey" "https://www.digikey.com/en/products/detail/walsin-technology-corporation/0603B103K500CT/9354883" (id 4) (at 135.89 59.69 0)
+      (effects (font (size 1.27 1.27)) hide)
+    )
