File: PC209/pulse_generator.kicad_sch (KiCad schematic)
At the start: 33 parts, among them Q10 BC848W, Q11 BC848W, Q12 BC848W, Q13 BC848W, Q14 BC848W, Q15 BC848W, Q2 BC848W

Commit message: PC209: Add BOM
Parts:
- C1, C5, R2, R22, R23, R28: Digikey (none) -> https://www.digikey.com/en/products/detail/walsin-technolog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
- C3, C4, C6, C7: Digikey (none) -> https://www.digikey.com/en/products/detail/samsung-electro-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
- Q10, Q11, Q12, Q13, Q14, Q15, Q2: Digikey (none) -> https://www.digikey.com/en/products/detail/nexperia-usa-inc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
- R11, R20, R21, R24, R25, R26, R27, R29, R30, R33, R34, R9: Digikey (none) -> https://www.digikey.com/en/products/detail/stackpole-electr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
Changed lines of the file:
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@@
+      (effects (font (size 1.27 1.27)) hide)
+    )
+    (property "Digikey" "https://www.digikey.com/en/products/detail/walsin-technology-corporation/WR06X3301FTL/13239039" (id 4) (at 124.46 100.33 0)
       (effects (font (size 1.27 1.27)) hide)
     )
@@
       (effects (font (size 1.27 1.27)) hide)
     )
+    (property "Digikey" "https://www.digikey.com/en/products/detail/samsung-electro-mechanics/CL10B471KB8NNNC/3886752" (id 4) (at 144.78 52.07 0)
+      (effects (font (size 1.27 1.27)) hide)
+    )
     (pin "1")
     (pin "2")
@@
       (effects (font (size 1.27 1.27)) hide)
     )
+    (property "Digikey" "https://www.digikey.com/en/products/detail/stackpole-electronics-inc/RMCF0603FT453R/1714054" (id 4) (at 171.45 48.26 0)
+      (effects (font (size 1.27 1.27)) hide)
+    )
     (pin "1")
     (pin "2")
@@
     (property "Datasheet" "http://www.infineon.com/dgdl/Infineon-BC847SERIES_BC848SERIES_BC849SERIES_BC850SERIES-DS-v01_01-en.pdf?fileId=db3a304314dca389011541d4630a1657" (id 3) (at 181.61 48.26 0)
       (effects (font (size 1.27 1.27)) (justify left) hide)
+    )
+    (property "Digikey" "https://www.digikey.com/en/products/detail/nexperia-usa-inc/BC848W-115/1232299" (id 4) (at 181.61 48.26 0)
+      (effects (font (size 1.27 1.27)) hide)
     )
     (pin "1")
@@
       (effects (font (size 1.27 1.27)) hide)
     )
+    (property "Digikey" "https://www.digikey.com/en/products/detail/stackpole-electronics-inc/RMCF0603FT634R/1760903" (id 4) (at 184.15 38.1 0)
+      (effects (font (size 1.27 1.27)) hide)
+    )
     (pin "1")
     (pin "2")
@@
       (effects (font (size 1.27 1.27)) hide)
     )
+    (property "Digikey" "https://www.digikey.com/en/products/detail/walsin-technology-corporation/0603B102K500CT/9354877" (id 4) (at 91.44 57.15 0)
+      (effects (font (size 1.27 1.27)) hide)
+    )
     (pin "1")
     (pin "2")
@@
       (effects (font (size 1.27 1.27)) hide)
     )
+    (property "Digikey" "https://www.digikey.com/en/products/detail/walsin-technology-corporation/WR06X102-JTL/13241138" (id 4) (at 97.79 63.5 0)
+      (effects (font (size 1.27 1.27)) hide)
+    )
     (pin "1")
     (pin "2")
@@
       (effects (font (size 1.27 1.27)) hide)
     )
+    (property "Digikey" "https://www.digikey.com/en/products/detail/stackpole-electronics-inc/RMCF0603FT453R/1714054" (id 4) (at 68.58 119.38 0)
+      (effects (font (size 1.27 1.27)) hide)
+    )
     (pin "1")
     (pin "2")
@@
     (property "Datasheet" "http://www.infineon.com/dgdl/Infineon-BC847SERIES_BC848SERIES_BC849SERIES_BC850SERIES-DS-v01_01-en.pdf?fileId=db3a304314dca389011541d4630a1657" (id 3) (at 88.9 119.38 0)
       (effects (font (size 1.27 1.27)) (justify left) hide)
+    )
+    (property "Digikey" "https://www.digikey.com/en/products/detail/nexperia-usa-inc/BC848W-115/1232299" (id 4) (at 88.9 119.38 0)
+      (effects (font (size 1.27 1.27)) hide)
     )
     (pin "1")
@@
       (effects (font (size 1.27 1.27)) hide)
     )
+    (property "Digikey" "https://www.digikey.com/en/products/detail/stackpole-electronics-inc/RMCF0603FT453R/1714054" (id 4) (at 99.06 119.38 0)
+      (effects (font (size 1.27 1.27)) hide)
+    )
     (pin "1")
     (pin "2")
@@
     (property "Datasheet" "http://www.infineon.com/dgdl/Infineon-BC847SERIES_BC848SERIES_BC849SERIES_BC850SERIES-DS-v01_01-en.pdf?fileId=db3a304314dca389011541d4630a1657" (id 3) (at 119.38 57.15 0)
       (effects (font (size 1.27 1.27)) (justify left) hide)
+    )
+    (property "Digikey" "https://www.digikey.com/en/products/detail/nexperia-usa-inc/BC848W-115/1232299" (id 4) (at 119.38 57.15 0)
+      (effects (font (size 1.27 1.27)) hide)
     )
     (pin "1")
@@
       (effects (font (size 1.27 1.27)) (justify left) hide)
     )
+    (property "Digikey" "https://www.digikey.com/en/products/detail/nexperia-usa-inc/BC848W-115/1232299" (id 4) (at 64.77 63.5 0)
+      (effects (font (size 1.27 1.27)) hide)
+    )
     (pin "1")
     (pin "2")
@@
     )
     (property "Datasheet" "~" (id 3) (at 139.7 57.15 0)
+      (effects (font (size 1.27 1.27)) hide)
+    )
+    (property "Digikey" "https://www.digikey.com/en/products/detail/stackpole-electronics-inc/RMCF0603FT453R/1714054" (id 4) (at 139.7 57.15 0)
       (effects (font (size 1.27 1.27)) hide)
     )
@@
       (effects (font (size 1.27 1.27)) hide)
     )
+    (property "Digikey" "https://www.digikey.com/en/products/detail/stackpole-electronics-inc/RMCF0603FT634R/1760903" (id 4) (at 143.51 100.33 0)
+      (effects (font (size 1.27 1.27)) hide)
+    )
     (pin "1")
     (pin "2")
@@
       (effects (font (size 1.27 1.27)) hide)
     )
+    (property "Digikey" "https://www.digikey.com/en/products/detail/stackpole-electronics-inc/RMCF0603FT634R/1760903" (id 4) (at 83.82 105.41 0)
+      (effects (font (size 1.27 1.27)) hide)
+    )
     (pin "1")
     (pin "2")
@@
       (effects (font (size 1.27 1.27)) hide)
     )
+    (property "Digikey" "https://www.digikey.com/en/products/detail/stackpole-electronics-inc/RMCF0603FT634R/1760903" (id 4) (at 67.31 53.34 0)
+      (effects (font (size 1.27 1.27)) hide)
+    )
     (pin "1")
     (pin "2")
@@
       (effects (font (size 1.27 1.27)) hide)
     )
+    (property "Digikey" "https://www.digikey.com/en/products/detail/stackpole-electronics-inc/RMCF0603FT634R/1760903" (id 4) (at 124.46 43.18 0)
+      (effects (font (size 1.27 1.27)) hide)
+    )
     (pin "1")
     (pin "2")
@@
       (effects (font (size 1.27 1.27)) hide)
     )
+    (property "Digikey" "https://www.digikey.com/en/products/detail/stackpole-electronics-inc/RMCF0603FT453R/1714054" (id 4) (at 109.22 57.15 0)
+      (effects (font (size 1.27 1.27)) hide)
+    )
     (pin "1")
     (pin "2")
@@
       (effects (font (size 1.27 1.27)) hide)
     )
+    (property "Digikey" "https://www.digikey.com/en/products/detail/walsin-technology-corporation/WR06X102-JTL/13241138" (id 4) (at 63.5 124.46 0)
+      (effects (font (size 1.27 1.27)) hide)
+    )
     (pin "1")
     (pin "2")
@@
     (property "Datasheet" "http://www.infineon.com/dgdl/Infineon-BC847SERIES_BC848SERIES_BC849SERIES_BC850SERIES-DS-v01_01-en.pdf?fileId=db3a304314dca389011541d4630a1657" (id 3) (at 129.54 57.15 0)
       (effects (font (size 1.27 1.27)) (justify left) hide)
+    )
+    (property "Digikey" "https://www.digikey.com/en/products/detail/nexperia-usa-inc/BC848W-115/1232299" (id 4) (at 129.54 57.15 0)
+      (effects (font (size 1.27 1.27)) hide)
     )
     (pin "1")
@@
     )
     (property "Datasheet" "~" (id 3) (at 165.1 38.1 0)
+      (effects (font (size 1.27 1.27)) hide)
+    )
+    (property "Digikey" "https://www.digikey.com/en/products/detail/walsin-technology-corporation/WR06X3301FTL/13239039" (id 4) (at 165.1 38.1 0)
       (effects (font (size 1.27 1.27)) hide)
     )
@@
       (effects (font (size 1.27 1.27)) (justify left) hide)
     )
+    (property "Digikey" "https://www.digikey.com/en/products/detail/nexperia-usa-inc/BC848W-115/1232299" (id 4) (at 78.74 119.38 0)
+      (effects (font (size 1.27 1.27)) hide)
+    )
     (pin "1")
     (pin "2")
@@
       (effects (font (size 1.27 1.27)) hide)
     )
+    (property "Digikey" "https://www.digikey.com/en/products/detail/stackpole-electronics-inc/RMCF0603FT453R/1714054" (id 4) (at 130.81 110.49 0)
+      (effects (font (size 1.27 1.27)) hide)
+    )
     (pin "1")
     (pin "2")
@@
     (property "Datasheet" "http://www.infineon.com/dgdl/Infineon-BC847SERIES_BC848SERIES_BC849SERIES_BC850SERIES-DS-v01_01-en.pdf?fileId=db3a304314dca389011541d4630a1657" (id 3) (at 140.97 110.49 0)
       (effects (font (size 1.27 1.27)) (justify left) hide)
+    )
+    (property "Digikey" "https://www.digikey.com/en/products/detail/nexperia-usa-inc/BC848W-115/1232299" (id 4) (at 140.97 110.49 0)
+      (effects (font (size 1.27 1.27)) hide)
     )
     (pin "1")
@@
       (effects (font (size 1.27 1.27)) hide)
     )
+    (property "Digikey" "https://www.digikey.com/en/products/detail/walsin-technology-corporation/0603B102K500CT/9354877" (id 4) (at 58.42 119.38 0)
+      (effects (font (size 1.27 1.27)) hide)
+    )
     (pin "1")
     (pin "2")
@@
       (effects (font (size 1.27 1.27)) hide)
     )
+    (property "Digikey" "https://www.digikey.com/en/products/detail/stackpole-electronics-inc/RMCF0603FT453R/1714054" (id 4) (at 54.61 63.5 0)
+      (effects (font (size 1.27 1.27)) hide)
+    )
     (pin "1")
     (pin "2")
@@
       (effects (font (size 1.27 1.27)) hide)
     )
+    (property "Digikey" "https://www.digikey.com/en/products/detail/samsung-electro-mechanics/CL10B104KB8NNWC/3887593" (id 4) (at 118.11 110.49 0)
+      (effects (font (size 1.27 1.27)) hide)
+    )
     (pin "1")
     (pin "2")
@@
       (effects (font (size 1.27 1.27)) hide)
     )
+    (property "Digikey" "https://www.digikey.com/en/products/detail/samsung-electro-mechanics/CL10B332KB8NNNC/3887416" (id 4) (at 158.75 48.26 0)
+      (effects (font (size 1.27 1.27)) hide)
+    )
     (pin "1")
     (pin "2")
@@
       (effects (font (size 1.27 1.27)) hide)
     )
+    (property "Digikey" "https://www.digikey.com/en/products/detail/samsung-electro-mechanics/CL10B471KB8NNNC/3886752" (id 4) (at 104.14 114.3 0)
+      (effects (font (size 1.27 1.27)) hide)
+    )
